File: pcb/rattlemebones32/rattlemebones32.kicad_pcb (KiCad board)
At the start: 2 copper layers, 171.4 x 76.5 mm, 85 parts, among them J1 USB_C_Receptacle_USB2.0, SW1 SW_Push, SW10 SW_Push, SW11 SW_Push, SW12 SW_Push, SW13 SW_Push, SW14 SW_Push, SW15 SW_Push, SW16 SW_Push, SW17 SW_Push, SW18 SW_Push, SW19 SW_Push, SW2 SW_Push, SW20 SW_Push, SW21 SW_Push, SW22 SW_Push, SW23 SW_Push, SW24 SW_Push, SW25 SW_Push, SW26 SW_Push, SW27 SW_Push, SW28 SW_Push, SW29 SW_Push, SW3 SW_Push, SW30 SW_Push, SW31 SW_Push, SW32 SW_Push, SW33 BOOT, SW34 RESET, SW4 SW_Push, SW5 SW_Push, SW6 SW_Push, SW7 SW_Push, SW8 SW_Push, SW9 SW_Push, U1 CH552T

Commit message: exports and case init
Parts:
- H1, H10, H11, H12, H2, H3, H4, H5, H6, H7, H8, H9: moved to B.Cu
- moved H8 173.1 mm to (171.9, 103.6), turned to -165 degrees
- moved H7 171.7 mm to (157.4, 107.5), turned to -165 degrees
- moved H6 164.6 mm to (193.1, 66.9), turned to -165 degrees
- moved SW33 151.9 mm to (120.3, 106.1), turned to -90 degrees
- moved H12 149.2 mm to (138.4, 106.4), turned to -165 degrees
- moved H4 147.0 mm to (93.2, 107.5), turned to 165 degrees
- moved SW34 146.2 mm to (130.3, 106.1), turned to -90 degrees
- moved H11 143.4 mm to (112.2, 106.4), turned to 165 degrees
- moved H5 142.9 mm to (149.6, 78.5), turned to -165 degrees
- moved H3 130.9 mm to (78.7, 103.6), turned to 165 degrees
- moved R1 130.2 mm to (116.6, 105.8), turned to -90 degrees
- moved H10 129.2 mm to (130.7, 77.4), turned to -165 degrees
- moved H2 119.1 mm to (101.0, 78.5), turned to 165 degrees
- moved H9 117.4 mm to (119.9, 77.4), turned to 165 degrees
- moved U1 110.7 mm to (125.3, 89.1)
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Connections:
- SW1 pad 2: col1 -> col10
- SW10 pad 2: col10 -> col1
- SW11 pad 2: col5 -> col6
- SW12 pad 2: col6 -> col5
- SW13 pad 2: col2 -> col9
- SW14 pad 2: col9 -> col2
- SW15 pad 2: col3 -> col8
- SW16 pad 2: col8 -> col3
- SW17 pad 2: col4 -> col7
- SW18 pad 2: col7 -> col4
- SW19 pad 2: col5 -> col6
- SW2 pad 2: col10 -> col1
- SW20 pad 2: col6 -> col5
- SW21 pad 2: col3 -> col8
- SW22 pad 2: col8 -> col3
- SW23 pad 2: col4 -> col7
- SW24 pad 2: col7 -> col4
- SW25 pad 2: col5 -> col6
- SW26 pad 2: col6 -> col5
- SW27 pad 2: col3 -> col8
- SW28 pad 2: col8 -> col3
- SW29 pad 2: col4 -> col7
- SW3 pad 2: col2 -> col9
- SW30 pad 2: col7 -> col4
- SW31 pad 2: col5 -> col6
- SW32 pad 2: col6 -> col5
- SW4 pad 2: col9 -> col2
- SW5 pad 2: col3 -> col8
- SW6 pad 2: col8 -> col3
- SW7 pad 2: col4 -> col7
- SW8 pad 2: col7 -> col4
- SW9 pad 2: col1 -> col10
Routing:
- net (no net): track 654.4 -> 0.00 mm
- net GND: track 0.00 -> 346.5 mm, vias 0 -> 4
- net row2: track 0.00 -> 203.2 mm, vias 0 -> 12
- net row1: track 0.00 -> 198.9 mm, vias 0 -> 12
- net row4: track 0.00 -> 170.2 mm, vias 0 -> 9
- net row3: track 0.00 -> 162.3 mm, vias 0 -> 11
- net col1: track 0.00 -> 114.4 mm, vias 0 -> 2
- net col3: track 0.00 -> 96.9 mm, vias 0 -> 2
- net col8: track 0.00 -> 92.7 mm, vias 0 -> 2
- net col10: track 0.00 -> 91.7 mm, vias 0 -> 2
- net col4: track 0.00 -> 82.3 mm, vias 0 -> 2
- net col2: track 0.00 -> 80.4 mm, vias 0 -> 2
- net col7: track 0.00 -> 80.2 mm
- net col9: track 0.00 -> 76.2 mm, vias 0 -> 2
- net col5: track 0.00 -> 67.7 mm
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Other:
- board text added: "rattlemebonez32 by sporewoh v0.0"
- board text added: "あなたはすでに骨になっています"
