File: pcb/rattlemebones32/rattlemebones32.kicad_sch (KiCad schematic)
At the start: 85 parts, among them J1 USB_C_Receptacle_USB2.0, SW1 BOOT, SW1 SW_Push, SW10 SW_Push, SW11 SW_Push, SW12 SW_Push, SW13 SW_Push, SW14 SW_Push, SW15 SW_Push, SW16 SW_Push, SW17 SW_Push, SW18 SW_Push, SW19 SW_Push, SW2 RESET, SW2 SW_Push, SW20 SW_Push, SW21 SW_Push, SW22 SW_Push, SW23 SW_Push, SW24 SW_Push, SW25 SW_Push, SW26 SW_Push, SW27 SW_Push, SW28 SW_Push, SW29 SW_Push, SW3 SW_Push, SW30 SW_Push, SW31 SW_Push, SW32 SW_Push, SW4 SW_Push, SW5 SW_Push, SW6 SW_Push, SW7 SW_Push, SW8 SW_Push, SW9 SW_Push, U1 CH552T

Commit message: exports and case init
Connections:
- net col1: now also SW10.2, SW2.2; no longer SW1.2, SW9.2
- net col10: now also SW1.2, SW9.2; no longer SW10.2, SW2.2
- net col2: now also SW14.2, SW4.2; no longer SW13.2, SW3.2
- net col3: now also SW16.2, SW22.2, SW28.2, SW6.2; no longer SW15.2, SW21.2, SW27.2, SW5.2
- net col4: now also SW18.2, SW24.2, SW30.2, SW8.2; no longer SW17.2, SW23.2, SW29.2, SW7.2
- net col5: now also SW12.2, SW20.2, SW26.2, SW32.2; no longer SW11.2, SW19.2, SW25.2, SW31.2
- net col6: now also SW11.2, SW19.2, SW25.2, SW31.2; no longer SW12.2, SW20.2, SW26.2, SW32.2
- net col7: now also SW17.2, SW23.2, SW29.2, SW7.2; no longer SW18.2, SW24.2, SW30.2, SW8.2
- net col8: now also SW15.2, SW21.2, SW27.2, SW5.2; no longer SW16.2, SW22.2, SW28.2, SW6.2
- net col9: now also SW13.2, SW3.2; no longer SW14.2, SW4.2
Changed lines of the file:
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@@
     (stroke (width 0) (type default))
   )
-  (global_label "col4" (shape input) (at 92.71 106.68 0) (fields_autoplaced)
+  (global_label "col7" (shape input) (at 92.71 106.68 0) (fields_autoplaced)
     (effects (font (size 1.27 1.27)) (justify left))
     (property "Intersheetrefs" "${INTERSHEET_REFS}" (at 99.8075 106.68 0)
@@
     )
   )
-  (global_label "col1" (shape input) (at 50.8 106.68 0) (fields_autoplaced)
-    (effects (font (size 1.27 1.27)) (justify left))
-    (property "Intersheetrefs" "${INTERSHEET_REFS}" (at 57.8975 106.68 0)
+  (global_label "col10" (shape input) (at 50.8 106.68 0) (fields_autoplaced)
+    (effects (font (size 1.27 1.27)) (justify left))
+    (property "Intersheetrefs" "${INTERSHEET_REFS}" (at 59.107 106.68 0)
       (effects (font (size 1.27 1.27)) (justify left) hide)
     )
@@
     )
   )
-  (global_label "col3" (shape input) (at 78.74 106.68 0) (fields_autoplaced)
+  (global_label "col8" (shape input) (at 78.74 106.68 0) (fields_autoplaced)
     (effects (font (size 1.27 1.27)) (justify left))
     (property "Intersheetrefs" "${INTERSHEET_REFS}" (at 85.8375 106.68 0)
@@
     )
   )
-  (global_label "col9" (shape input) (at 161.29 106.68 0) (fields_autoplaced)
+  (global_label "col2" (shape input) (at 161.29 106.68 0) (fields_autoplaced)
     (effects (font (size 1.27 1.27)) (justify left))
     (property "Intersheetrefs" "${INTERSHEET_REFS}" (at 168.3875 106.68 0)
@@
     )
   )
-  (global_label "col5" (shape input) (at 105.41 106.68 0) (fields_autoplaced)
+  (global_label "col6" (shape input) (at 105.41 106.68 0) (fields_autoplaced)
     (effects (font (size 1.27 1.27)) (justify left))
     (property "Intersheetrefs" "${INTERSHEET_REFS}" (at 112.5075 106.68 0)
@@
     )
   )
-  (global_label "col2" (shape input) (at 64.77 106.68 0) (fields_autoplaced)
+  (global_label "col9" (shape input) (at 64.77 106.68 0) (fields_autoplaced)
     (effects (font (size 1.27 1.27)) (justify left))
     (property "Intersheetrefs" "${INTERSHEET_REFS}" (at 71.8675 106.68 0)
@@
     )
   )
-  (global_label "col7" (shape input) (at 133.35 106.68 0) (fields_autoplaced)
+  (global_label "col4" (shape input) (at 133.35 106.68 0) (fields_autoplaced)
     (effects (font (size 1.27 1.27)) (justify left))
     (property "Intersheetrefs" "${INTERSHEET_REFS}" (at 140.4475 106.68 0)
@@
     )
   )
-  (global_label "col10" (shape input) (at 175.26 106.68 0) (fields_autoplaced)
-    (effects (font (size 1.27 1.27)) (justify left))
-    (property "Intersheetrefs" "${INTERSHEET_REFS}" (at 183.567 106.68 0)
+  (global_label "col1" (shape input) (at 175.26 106.68 0) (fields_autoplaced)
+    (effects (font (size 1.27 1.27)) (justify left))
+    (property "Intersheetrefs" "${INTERSHEET_REFS}" (at 182.3575 106.68 0)
       (effects (font (size 1.27 1.27)) (justify left) hide)
     )
@@
     )
   )
-  (global_label "col6" (shape input) (at 119.38 106.68 0) (fields_autoplaced)
+  (global_label "col5" (shape input) (at 119.38 106.68 0) (fields_autoplaced)
     (effects (font (size 1.27 1.27)) (justify left))
     (property "Intersheetrefs" "${INTERSHEET_REFS}" (at 126.4775 106.68 0)
@@
     )
   )
-  (global_label "col8" (shape input) (at 147.32 106.68 0) (fields_autoplaced)
+  (global_label "col3" (shape input) (at 147.32 106.68 0) (fields_autoplaced)
     (effects (font (size 1.27 1.27)) (justify left))
     (property "Intersheetrefs" "${INTERSHEET_REFS}" (at 154.4175 106.68 0)
